Commit message: removed prefix args

File: ur_description/urdf/ur10_robot.urdf.xacro (robot description, xacro)
@@ -7,9 +7,9 @@
   <xacro:include filename="$(find ur_description)/urdf/ur10.urdf.xacro" />
   <!-- arm -->
-  <xacro:ur10_robot prefix="$(arg prefix)" joint_limited="$(arg limited)"/>
+  <xacro:ur10_robot prefix="" joint_limited="$(arg limited)"/>
   <link name="world" />
   <joint name="world_joint" type="fixed">
     <parent link="world" />
-    <child link = "$(arg prefix)base_link" />
+    <child link = "base_link" />
     <origin xyz="0.0 0.0 0.0" rpy="0.0 0.0 0.0" />
   </joint>

File: ur_description/urdf/ur3_robot.urdf.xacro (robot description, xacro)
@@ -7,9 +7,9 @@
   <xacro:include filename="$(find ur_description)/urdf/ur3.urdf.xacro" />
   <!-- arm -->
-  <xacro:ur3_robot prefix="$(arg prefix)" joint_limited="$(arg limited)"/>
+  <xacro:ur3_robot prefix="" joint_limited="$(arg limited)"/>
   <link name="world" />
   <joint name="world_joint" type="fixed">
     <parent link="world" />
-    <child link = "$(arg prefix)base_link" />
+    <child link = "base_link" />
     <origin xyz="0.0 0.0 0.0" rpy="0.0 0.0 0.0" />
   </joint>

File: ur_description/urdf/ur5_robot.urdf.xacro (robot description, xacro)
@@ -7,9 +7,9 @@
   <xacro:include filename="$(find ur_description)/urdf/ur5.urdf.xacro" />
   <!-- arm -->
-  <xacro:ur5_robot prefix="$(arg prefix)" joint_limited="$(arg limited)"/>
+  <xacro:ur5_robot prefix="" joint_limited="$(arg limited)"/>
   <link name="world" />
   <joint name="world_joint" type="fixed">
     <parent link="world" />
-    <child link = "$(arg prefix)base_link" />
+    <child link = "base_link" />
     <origin xyz="0.0 0.0 0.0" rpy="0.0 0.0 0.0" />
   </joint>
